Commit message: Task 2.03 - Added fixed URDF files

File: urdf_package/urdf/Part1.urdf (robot description, URDF)
Before this commit: robot Part1, 1 links, 0 joints
Links:
- removed link turtlebot_world
- added link urdf_package, mass 5806.9; collision mesh filename=package://urdf_package/meshes/turtlebot_world_col.STL; visual mesh filename=package://urdf_package/meshes/turtlebot_world.STL
