Commit message: Task 3.13 - [kobuki.urdf.xacro] Adding additional link to keep scooper from being too deep

File: urdf_package/modifiedKobuki/kobuki.urdf.xacro (robot description, xacro)
@@ -29,5 +29,5 @@
       <pose frame=''>-0 -0 0 0 -0 0</pose>
       <inertial>
-<mass value="1.0"/>
+<mass value="0.1"/>
         <inertia ixx="0.166667" ixy="0.0" ixz="0.0"
                  iyy="0.166667" iyz="0.0"
@@ -105,8 +105,8 @@
       <child link="leftScoop" />
     </joint>
-<link name='rightScoop'>
+    <link name='middleScoop'>
       <pose frame=''>-0 -0 0 0 -0 0</pose>
       <inertial>
-<mass value="1.0"/>
+<mass value="0.1"/>
         <inertia ixx="0.166667" ixy="0.0" ixz="0.0"
                  iyy="0.166667" iyz="0.0"
@@ -120,5 +120,5 @@
         <pose frame=''>0 0 0 0 -0 0</pose>
         <geometry>
-          <box size="0.5 0.1 0.1"/>
+          <box size="0.2 0.1 0.1"/>
         </geometry>
         <cast_shadows>1</cast_shadows>
@@ -130,5 +130,5 @@
         <pose frame=''>0 0 0 0 -0 0</pose>
         <geometry>
-<box size="0.5 0.1 0.1"/>
+<box size="0.2 0.1 0.1"/>
         </geometry>
         <surface>
@@ -180,4 +180,83 @@
     </link>
     <joint name="base_joint3" type="fixed">
+      <origin xyz="0.23 0.0 0.1" rpy="0 0 1.571" />
+      <parent link="base_footprint"/>
+      <child link="middleScoop" />
+    </joint>
+<link name='rightScoop'>
+      <pose frame=''>-0 -0 0 0 -0 0</pose>
+      <inertial>
+<mass value="0.1"/>
+        <inertia ixx="0.166667" ixy="0.0" ixz="0.0"
+                 iyy="0.166667" iyz="0.0"
+                 izz="0.166667" />
+      </inertial>
+        <pose frame=''>0 0 0 0 -0 0</pose>
+      <gravity>1</gravity>
+      <self_collide>0</self_collide>
+      <kinematic>0</kinematic>
+      <visual name='visual'>
+        <pose frame=''>0 0 0 0 -0 0</pose>
+        <geometry>
+          <box size="0.5 0.1 0.1"/>
+        </geometry>
+        <cast_shadows>1</cast_shadows>
+        <transparency>0</transparency>
+      </visual>
+      <collision name='collision'>
+        <laser_retro>0</laser_retro>
+        <max_contacts>10</max_contacts>
+        <pose frame=''>0 0 0 0 -0 0</pose>
+        <geometry>
+<box size="0.5 0.1 0.1"/>
+        </geometry>
+        <surface>
+          <friction>
+            <ode>
+              <mu>1</mu>
+              <mu2>1</mu2>
+              <fdir1>0 0 0</fdir1>
+              <slip1>0</slip1>
+              <slip2>0</slip2>
+            </ode>
+            <torsional>
+              <coefficient>1</coefficient>
+              <patch_radius>0</patch_radius>
+              <surface_radius>0</surface_radius>
+              <use_patch_radius>1</use_patch_radius>
+              <ode>
+                <slip>0</slip>
+              </ode>
+            </torsional>
+          </friction>
+          <bounce>
+            <restitution_coefficient>0</restitution_coefficient>
+            <threshold>1e+06</threshold>
+          </bounce>
+          <contact>
+            <collide_without_contact>0</collide_without_contact>
+            <collide_without_contact_bitmask>1</collide_without_contact_bitmask>
+            <collide_bitmask>1</collide_bitmask>
+            <ode>
+              <soft_cfm>0</soft_cfm>
+              <soft_erp>0.2</soft_erp>
+              <kp>1e+13</kp>
+              <kd>1</kd>
+              <max_vel>0.01</max_vel>
+              <min_depth>0</min_depth>
+            </ode>
+            <bullet>
+              <split_impulse>1</split_impulse>
+              <split_impulse_penetration_threshold>-0.01</split_impulse_penetration_threshold>
+              <soft_cfm>0</soft_cfm>
+              <soft_erp>0.2</soft_erp>
+              <kp>1e+13</kp>
+              <kd>1</kd>
+            </bullet>
+          </contact>
+        </surface>
+      </collision>
+    </link>
+    <joint name="base_joint4" type="fixed">
       <origin xyz="0.2 -0.2 0.1" rpy="0 0 0.2" />
       <parent link="base_footprint"/>
